Commit message: Update lidar.xacro

File: src/main_sim/urdf/lidar.xacro (robot description, xacro)
@@ -1,10 +1,11 @@
 <?xml version="1.0"?>
-<robot xmlns:xacro="http://www.ros.org/wiki/xacro">
+<robot xmlns:xacro="http://www.ros.org/xacro">
+    <!-- Lidar Joint -->
     <joint name="laser_joint" type="fixed">
         <parent link="chassis"/>
         <child link="laser_frame"/>
-        <!-- puts origin of laser link on top of robot -->
         <origin xyz="0.1 0 0.175" rpy="0 0 0"/>
     </joint>
+    <!-- Lidar Frame -->
     <link name="laser_frame">
         <visual>
@@ -23,50 +24,16 @@
         </xacro:inertial_cylinder>
     </link>
-    <!-- Gazebo Tag -->
-    <gazebo reference="laser_frame">
-        <material>Gazebo/Red</material>
-        <sensor name="laser" type="ray">
-            <pose> 0 0 0 0 0 0 </pose>
-            <!-- visualize in gazebo -->
-            <visualize>false</visualize>
-            <!-- 10 updates a second -->
-            <update_rate>10</update_rate>
-            <!-- parameters for lidar sensor -->
-            <ray>
-                <scan>
-                    <horizontal>
-                        <!-- resolution of 1 (1 degree of error) -->
-                        <samples>360</samples>
-                        <min_angle>-3.14</min_angle>
-                        <max_angle>3.14</max_angle>
-                    </horizontal>
-                </scan>
-                <range>
-                    <min>0.3</min>
-                    <max>12</max>
-                </range>
-            </ray>
-            <!-- Plugin that takes ray sensor and gets it to publish data to the scan topic -->
-            <plugin name="laser_controller" filename="libgazebo_ros_ray_sensor.so">
-                <ros>
-                    <argument>~/out:=scan</argument>
-                </ros>
-                <output_type>sensor_msgs/LaserScan</output_type>
-                <frame_name>laser_frame</frame_name>
-            </plugin><visual>
-                <geometry>
-                    <cylinder radius="0.05" length="0.04"/>
-                </geometry>
-                <material name="blue"/>
-            </visual>
-            <collision>
-                <geometry>
-                    <cylinder radius="0.05" length="0.04"/>
-                </geometry>
-            </collision>
-            <xacro:inertial_cylinder mass="0.1" length="0.04" radius="0.05">
-                <origin xyz="0 0 0" rpy="0 0 0"/>
-            </xacro:inertial_cylinder>
-        </sensor>
+    <!-- Gazebo Sim (Ignition) Plugin -->
+    <gazebo>
+        <plugin name="gz_ros2_lidar" filename="libgz_ros2_lidar.so">
+            <param name="topic">/scan</param>
+            <param name="frame_name">laser_frame</param>
+            <param name="hz">10</param> <!-- Update rate -->
+            <param name="horizontal_samples">360</param>
+            <param name="horizontal_min_angle">-3.14</param>
+            <param name="horizontal_max_angle">3.14</param>
+            <param name="range_min">0.3</param>
+            <param name="range_max">12</param>
+        </plugin>
     </gazebo>
 </robot>

Commit message: Update lidar.xacro

File: src/main_sim/urdf/lidar.xacro (robot description, xacro)
@@ -1,11 +1,10 @@
 <?xml version="1.0"?>
-<robot xmlns:xacro="http://www.ros.org/xacro">
-    <!-- Lidar Joint -->
+<robot xmlns:xacro="http://www.ros.org/wiki/xacro">
     <joint name="laser_joint" type="fixed">
         <parent link="chassis"/>
         <child link="laser_frame"/>
+        <!-- puts origin of laser link on top of robot -->
         <origin xyz="0.1 0 0.175" rpy="0 0 0"/>
     </joint>
-    <!-- Lidar Frame -->
     <link name="laser_frame">
         <visual>
@@ -24,16 +23,50 @@
         </xacro:inertial_cylinder>
     </link>
-    <!-- Gazebo Sim (Ignition) Plugin -->
-    <gazebo>
-        <plugin name="gz_ros2_lidar" filename="libgz_ros2_lidar.so">
-            <param name="topic">/scan</param>
-            <param name="frame_name">laser_frame</param>
-            <param name="hz">10</param> <!-- Update rate -->
-            <param name="horizontal_samples">360</param>
-            <param name="horizontal_min_angle">-3.14</param>
-            <param name="horizontal_max_angle">3.14</param>
-            <param name="range_min">0.3</param>
-            <param name="range_max">12</param>
-        </plugin>
+    <!-- Gazebo Tag -->
+    <gazebo reference="laser_frame">
+        <material>Gazebo/Red</material>
+        <sensor name="laser" type="ray">
+            <pose> 0 0 0 0 0 0 </pose>
+            <!-- visualize in gazebo -->
+            <visualize>false</visualize>
+            <!-- 10 updates a second -->
+            <update_rate>10</update_rate>
+            <!-- parameters for lidar sensor -->
+            <ray>
+                <scan>
+                    <horizontal>
+                        <!-- resolution of 1 (1 degree of error) -->
+                        <samples>360</samples>
+                        <min_angle>-3.14</min_angle>
+                        <max_angle>3.14</max_angle>
+                    </horizontal>
+                </scan>
+                <range>
+                    <min>0.3</min>
+                    <max>12</max>
+                </range>
+            </ray>
+            <!-- Plugin that takes ray sensor and gets it to publish data to the scan topic -->
+            <plugin name="laser_controller" filename="libgazebo_ros_ray_sensor.so">
+                <ros>
+                    <argument>~/out:=scan</argument>
+                </ros>
+                <output_type>sensor_msgs/LaserScan</output_type>
+                <frame_name>laser_frame</frame_name>
+            </plugin><visual>
+                <geometry>
+                    <cylinder radius="0.05" length="0.04"/>
+                </geometry>
+                <material name="blue"/>
+            </visual>
+            <collision>
+                <geometry>
+                    <cylinder radius="0.05" length="0.04"/>
+                </geometry>
+            </collision>
+            <xacro:inertial_cylinder mass="0.1" length="0.04" radius="0.05">
+                <origin xyz="0 0 0" rpy="0 0 0"/>
+            </xacro:inertial_cylinder>
+        </sensor>
     </gazebo>
 </robot>

Commit message: migration finished

File: src/main_sim/urdf/lidar.xacro (robot description, xacro)
@@ -26,5 +26,5 @@
     <gazebo reference="laser_frame">
         <material>Gazebo/Red</material>
-        <sensor name="laser" type="ray">
+        <sensor name="laser" type="gpu_lidar">
             <pose> 0 0 0 0 0 0 </pose>
             <!-- visualize in gazebo -->
@@ -33,5 +33,5 @@
             <update_rate>10</update_rate>
             <!-- parameters for lidar sensor -->
-            <ray>
+            <lidar>
                 <scan>
                     <horizontal>
@@ -46,26 +46,7 @@
                     <max>12</max>
                 </range>
-            </ray>
-            <!-- Plugin that takes ray sensor and gets it to publish data to the scan topic -->
-            <plugin name="laser_controller" filename="libgazebo_ros_ray_sensor.so">
-                <ros>
-                    <argument>~/out:=scan</argument>
-                </ros>
-                <output_type>sensor_msgs/LaserScan</output_type>
-                <frame_name>laser_frame</frame_name>
-            </plugin><visual>
-                <geometry>
-                    <cylinder radius="0.05" length="0.04"/>
-                </geometry>
-                <material name="blue"/>
-            </visual>
-            <collision>
-                <geometry>
-                    <cylinder radius="0.05" length="0.04"/>
-                </geometry>
-            </collision>
-            <xacro:inertial_cylinder mass="0.1" length="0.04" radius="0.05">
-                <origin xyz="0 0 0" rpy="0 0 0"/>
-            </xacro:inertial_cylinder>
+            </lidar>
+                <topic>scan</topic>
+                <gz_frame_id>laser_frame</gz_frame_id>
         </sensor>
     </gazebo>

File: src/main_sim/urdf/ros2_control.xacro (robot description, xacro)
@@ -3,5 +3,5 @@
     <ros2_control name="GazeboSystem" type="system">
         <hardware>
-            <plugin>gazebo_ros2_control/GazeboSystem</plugin>
+            <plugin>gz_ros2_control/GazeboSimSystem</plugin>
         </hardware>
         <joint name="left_wheel_joint">
@@ -23,7 +23,7 @@
     </ros2_control>
     <gazebo>
-        <plugin name="gz_ros2_control" filename="libgazebo_ros2_control.so">
-            <param name="robot_description">robot_description</param>
-            <param name="use_sim_time">true</param>
+        <plugin name="gz_ros2_control::GazeboSimROS2ControlPlugin" filename="libgz_ros2_control-system.so">
+            <parameters>src/main_sim/config/my_controllers.yaml</parameters>
+            <parameters>/home/jason/ros2_ws/src/main_sim/config/ros_gz_ctrl_use_sim.yaml</parameters>
         </plugin>
     </gazebo>
