Commit message: Changes to be committed: 	modified:   build/main_sim/symlink_install_manifest.txt 	modified:   log/latest_build 	new file:   src/main_sim/launch/launch_mecanum.launch.py 	modified:   src/main_sim/urdf/mecanum_robot.urdf.xacro

File: src/main_sim/urdf/mecanum_robot.urdf.xacro (robot description, xacro)
@@ -1,197 +1,7 @@
-<?xml version="1.0" ?>
-<robot name="mecanumbot" xmlns:xacro="http://ros.org/wiki/xacro">
-  <material name="darkgrey">
-    <color rgba="0.1 0.1 0.1 1.0" />
-  </material>
-  <material name="grey">
-    <color rgba="0.5 0.5 0.5 1.0" />
-  </material>
-  <material name="blue">
-    <color rgba="0.0 0.0 0.8 1.0" />
-  </material>
-  <xacro:property name="M_PI" value="3.1415926535897931" />
-  <xacro:property name="M_PI_2" value="1.570796327" />
-  <xacro:property name="DEG_TO_RAD" value="0.017453293" />
-  <xacro:property name="base_size_x" value="0.44" />
-  <xacro:property name="base_size_y" value="0.40" />
-  <xacro:property name="base_size_z" value="0.02" />
-  <xacro:property name="base_mass" value="1.000" />
-  <xacro:property name="wheel_radius" value="0.03" />
-  <xacro:property name="wheel_width" value="0.03" />
-  <xacro:property name="wheel_offset_x" value="0.19"/>
-  <xacro:property name="wheel_offset_y" value="0.22"/>
-  <xacro:property name="wheel_offset_z" value="-0.03"/>
-  <xacro:property name="wheel_mass" value="0.500"/>
-  <xacro:macro name="box_inertia" params="m x y z">
-    <inertia ixx="${m*(y*y+z*z)/12}" ixy="0" ixz="0"
-             iyy="${m*(x*x+z*z)/12}" iyz="0"
-             izz="${m*(x*x+z*z)/12}"
-    />
-  </xacro:macro>
-  <xacro:macro name="cylinder_inertia" params="m r w">
-    <inertia ixx="${m*(3*r*r+w*w)/12}" ixy="0" ixz="0"
-             iyy="${m*(3*r*r+w*w)/12}" iyz="0"
-             izz="${m*r*r/2}"
-    />
-  </xacro:macro>
-  <link name="base_footprint" />
-  <joint name="base_joint" type="fixed">
-    <parent link="base_footprint" />
-    <child link="base_link" />
-    <origin xyz="0 0 0" rpy="0 0 0" />
-  </joint>
-  <link name="base_link">
-    <visual>
-      <origin xyz="0 0 0" rpy="0 0 0" />
-      <geometry>
-        <box size="${base_size_x} ${base_size_y} ${base_size_z}" />
-      </geometry>
-      <material name="grey" />
-    </visual>
-    <collision>
-      <origin xyz="0 0 0" rpy="0 0 0" />
-      <geometry>
-        <box size="${base_size_x} ${base_size_y} ${base_size_z}" />
-      </geometry>
-    </collision>
-    <inertial>
-      <origin xyz="0.0 0.0 0.0" rpy="0.0 0.0 0.0"/>
-      <mass value="${base_mass}"/>
-      <xacro:box_inertia m="${base_mass}" x="${base_size_x}" y="${base_size_y}" z="${base_size_z}"/>
-    </inertial>
-  </link>
-  <joint name="fl_wheel_joint" type="continuous">
-    <parent link="base_link"/>
-    <child link="fl_wheel_link"/>
-    <origin xyz="${-wheel_offset_x} ${-wheel_offset_y} ${wheel_offset_z}" rpy="0 0 ${-M_PI/2}" />
-    <axis xyz="1 0 0" rpy="0 0 0"/>
-  </joint>
-  <link name="fl_wheel_link">
-    <visual>
-      <origin xyz="0 0 0" rpy="0 0 0" />
-      <geometry>
-        <mesh filename="package://mecanumbot_description/meshes/fl_wheel_link.STL" scale="0.6 0.6 0.6" />
-      </geometry>
-      <material name="darkgrey" />
-    </visual>
-    <collision>
-      <origin xyz="0 0 0" rpy="0 0 0" />
-      <geometry>
-        <box size="${wheel_width} ${wheel_radius*2} ${wheel_radius*2}" />
-      </geometry>
-    </collision>
-    <inertial>
-      <origin xyz="0 0 0" rpy="0 0 0" />
-      <mass value="${wheel_mass}" />
-      <xacro:cylinder_inertia m="${wheel_mass}" r="${wheel_radius}" w="${wheel_width}" />
-    </inertial>
-  </link>
-  <joint name="fr_wheel_joint" type="continuous">
-    <parent link="base_link"/>
-    <child link="fr_wheel_link"/>
-    <origin xyz="${-wheel_offset_x} ${wheel_offset_y} ${wheel_offset_z}" rpy="0 0 ${M_PI/2}" />
-    <axis xyz="-1 0 0" rpy="0 0 0"/>
-  </joint>
-  <link name="fr_wheel_link">
-    <visual>
-      <origin xyz="0 0 0" rpy="0 0 0" />
-      <geometry>
-        <mesh filename="package://mecanumbot_description/meshes/fr_wheel_link.STL" scale="0.6 0.6 0.6" />
-      </geometry>
-      <material name="darkgrey" />
-    </visual>
-    <collision>
-      <origin xyz="0 0 0" rpy="0 0 0" />
-      <geometry>
-        <box size="${wheel_width} ${wheel_radius*2} ${wheel_radius*2}" />
-      </geometry>
-    </collision>
-    <inertial>
-      <origin xyz="0 0 0" rpy="0 0 0" />
-      <mass value="${wheel_mass}" />
-      <xacro:cylinder_inertia m="${wheel_mass}" r="${wheel_radius}" w="${wheel_width}" />
-    </inertial>
-  </link>
-  <joint name="rl_wheel_joint" type="continuous">
-    <parent link="base_link"/>
-    <child link="rl_wheel_link"/>
-    <origin xyz="${wheel_offset_x} ${-wheel_offset_y} ${wheel_offset_z}" rpy="0 0 ${-M_PI/2}" />
-    <axis xyz="1 0 0" rpy="0 0 0"/>
-  </joint>
-  <link name="rl_wheel_link">
-    <visual>
-      <origin xyz="0 0 0" rpy="0 0 0" />
-      <geometry>
-        <mesh filename="package://mecanumbot_description/meshes/rl_wheel_link.STL" scale="0.6 0.6 0.6" />
-      </geometry>
-      <material name="darkgrey" />
-    </visual>
-    <collision>
-      <origin xyz="0 0 0" rpy="0 0 0" />
-      <geometry>
-        <box size="${wheel_width} ${wheel_radius*2} ${wheel_radius*2}" />
-      </geometry>
-    </collision>
-    <inertial>
-      <origin xyz="0 0 0" rpy="0 0 0" />
-      <mass value="${wheel_mass}" />
-      <xacro:cylinder_inertia m="${wheel_mass}" r="${wheel_radius}" w="${wheel_width}" />
-    </inertial>
-  </link>
-  <joint name="rr_wheel_joint" type="continuous">
-    <parent link="base_link"/>
-    <child link="rr_wheel_link"/>
-    <origin xyz="${wheel_offset_x} ${wheel_offset_y} ${wheel_offset_z}" rpy="0 0 ${M_PI/2}" />
-    <axis xyz="-1 0 0" rpy="0 0 0"/>
-  </joint>
-  <link name="rr_wheel_link">
-    <visual>
-      <origin xyz="0 0 0" rpy="0 0 0" />
-      <geometry>
-        <mesh filename="package://mecanumbot_description/meshes/rr_wheel_link.STL" scale="0.6 0.6 0.6" />
-      </geometry>
-      <material name="darkgrey" />
-    </visual>
-    <collision>
-      <origin xyz="0 0 0" rpy="0 0 0" />
-      <geometry>
-        <box size="${wheel_width} ${wheel_radius*2} ${wheel_radius*2}" />
-      </geometry>
-    </collision>
-    <inertial>
-      <origin xyz="0 0 0" rpy="0 0 0" />
-      <mass value="${wheel_mass}" />
-      <xacro:cylinder_inertia m="${wheel_mass}" r="${wheel_radius}" w="${wheel_width}" />
-    </inertial>
-  </link>
-  <ros2_control name="mecanumbot" type="system">
-    <hardware>
-      <plugin>mecanumbot_hardware/MecanumbotHardware</plugin>
-      <param name="serial_port">/dev/ttyACM0</param>
-    </hardware>
-    <joint name="fl_wheel_joint">
-      <command_interface name="velocity" />
-      <state_interface name="position" />
-      <state_interface name="velocity" />
-      <param name="motor_id">1</param>
-    </joint>
-    <joint name="fr_wheel_joint">
-      <command_interface name="velocity" />
-      <state_interface name="position" />
-      <state_interface name="velocity" />
-      <param name="motor_id">2</param>
-    </joint>
-    <joint name="rl_wheel_joint">
-      <command_interface name="velocity" />
-      <state_interface name="position" />
-      <state_interface name="velocity" />
-      <param name="motor_id">4</param>
-    </joint>
-    <joint name="rr_wheel_joint">
-      <command_interface name="velocity" />
-      <state_interface name="position" />
-      <state_interface name="velocity" />
-      <param name="motor_id">8</param>
-    </joint>
-  </ros2_control>
+<?xml version="1.0"?>
+<robot xmlns:xacro="http://www.ros.org/wiki/xacro" name="robot">
+    <xacro:include filename="mecanum_core.xacro" />
+    <!-- <xacro:include filename="gazebo_control.xacro"/> -->
+    <xacro:include filename="mecanum_ros2_control.xacro"/>
+    <!-- <xacro:include filename="lidar.xacro"/> -->
 </robot>
