Commit message: Update mecanum_inertial_macros.xacro

File: src/main_sim/urdf/mecanum_inertial_macros.xacro (robot description, xacro)
@@ -1,5 +1,5 @@
 <?xml version="1.0"?>
 <robot xmlns:xacro="http://www.ros.org/xacro" >
-    <!-- Specify standard inertial calculations -->
+    <!-- Macro to define inertial properties for a box -->
     <xacro:macro name="inertial_box" params="mass x y z *origin">
         <inertial>
@@ -11,7 +11,14 @@
         </inertial>
     </xacro:macro>
+    <!-- Macro to define inertial properties for a cylinder -->
     <xacro:macro name="inertial_cylinder" params="mass length radius *origin">
         <inertial>
-            <xacro:insert_block name="origin"/>
+            <!-- Ensure an origin is always included -->
+            <xacro:if value="${origin}">
+                <xacro:insert_block name="origin"/>
+            </xacro:if>
+            <xacro:unless value="${origin}">
+                <origin xyz="0 0 0" rpy="0 0 0"/>
+            </xacro:unless>
             <mass value="${mass}" />
             <inertia ixx="${(1/12) * mass * (3*radius*radius + length*length)}" ixy="0.0" ixz="0.0"
