Commit message: Update mecanum_core.xacro

File: src/main_sim/urdf/mecanum_core.xacro (robot description, xacro)
@@ -2,15 +2,13 @@
 <robot xmlns:xacro="http://www.ros.org/xacro">
     <xacro:include filename="inertial_macros.xacro"/>
+    <!-- Define Materials -->
     <material name="white">
-        <color rgba="1 1 1 1" />
+        <color rgba="1 1 1 1"/>
     </material>
     <material name="blue">
         <color rgba="0.2 0.2 1 1"/>
     </material>
-    <material name="black">
-        <color rgba="0 0 0 1"/>
-    </material>
     <!-- BASE LINK -->
-    <link name="base_link"></link>
+    <link name="base_link"/>
     <!-- BASE_FOOTPRINT LINK -->
     <joint name="base_footprint_joint" type="fixed">
@@ -19,14 +17,14 @@
         <origin xyz="0 0 0" rpy="0 0 0"/>
     </joint>
-    <link name="base_footprint"></link>
-    <!-- CHASSIS LINK -->
+    <link name="base_footprint"/>
+    <!-- CHASSIS -->
     <joint name="chassis_joint" type="fixed">
         <parent link="base_link"/>
         <child link="chassis"/>
-        <origin xyz="-0.1 0 0"/>
+        <origin xyz="0 0 0"/>
     </joint>
     <link name="chassis">
         <visual>
-            <origin xyz="0.15 0 0.075"/>
+            <origin xyz="0 0 0.075"/>
             <geometry>
                 <box size="0.3 0.3 0.15"/>
@@ -35,5 +33,5 @@
         </visual>
         <collision>
-            <origin xyz="0.15 0 0.075"/>
+            <origin xyz="0 0 0.075"/>
             <geometry>
                 <box size="0.3 0.3 0.15"/>
@@ -41,15 +39,12 @@
         </collision>
         <xacro:inertial_box mass="0.5" x="0.3" y="0.3" z="0.15">
-            <origin xyz="0.15 0 0.075" rpy="0 0 0"/>
+            <origin xyz="0 0 0.075" rpy="0 0 0"/>
         </xacro:inertial_box>
     </link>
-    <gazebo reference="chassis">
-        <material>Gazebo/White</material>
-    </gazebo>
     <!-- FRONT LEFT WHEEL -->
     <joint name="front_left_wheel_joint" type="continuous">
         <parent link="base_link"/>
         <child link="front_left_wheel"/>
-        <origin xyz="0.15 0.15 0" rpy="-1.57079632679 0 0"/>
+        <origin xyz="0.15 0.15 0.05" rpy="0 0 0"/>
         <axis xyz="0 0 1"/>
     </joint>
@@ -66,7 +61,5 @@
             </geometry>
         </collision>
-        <xacro:inertial_cylinder mass="0.1" length="0.04" radius="0.05">
-            <origin xyz="0 0 0" rpy="0 0 0"/>
-        </xacro:inertial_cylinder>
+        <xacro:inertial_cylinder mass="0.1" length="0.04" radius="0.05"/>
     </link>
     <!-- FRONT RIGHT WHEEL -->
@@ -74,5 +67,5 @@
         <parent link="base_link"/>
         <child link="front_right_wheel"/>
-        <origin xyz="0.15 -0.15 0" rpy="1.57079632679 0 0"/>
+        <origin xyz="0.15 -0.15 0.05" rpy="0 0 0"/>
         <axis xyz="0 0 -1"/>
     </joint>
@@ -89,7 +82,5 @@
             </geometry>
         </collision>
-        <xacro:inertial_cylinder mass="0.1" length="0.04" radius="0.05">
-            <origin xyz="0 0 0" rpy="0 0 0"/>
-        </xacro:inertial_cylinder>
+        <xacro:inertial_cylinder mass="0.1" length="0.04" radius="0.05"/>
     </link>
     <!-- REAR LEFT WHEEL -->
@@ -97,5 +88,5 @@
         <parent link="base_link"/>
         <child link="rear_left_wheel"/>
-        <origin xyz="-0.15 0.15 0" rpy="-1.57079632679 0 0"/>
+        <origin xyz="-0.15 0.15 0.05" rpy="0 0 0"/>
         <axis xyz="0 0 1"/>
     </joint>
@@ -112,7 +103,5 @@
             </geometry>
         </collision>
-        <xacro:inertial_cylinder mass="0.1" length="0.04" radius="0.05">
-            <origin xyz="0 0 0" rpy="0 0 0"/>
-        </xacro:inertial_cylinder>
+        <xacro:inertial_cylinder mass="0.1" length="0.04" radius="0.05"/>
     </link>
     <!-- REAR RIGHT WHEEL -->
@@ -120,5 +109,5 @@
         <parent link="base_link"/>
         <child link="rear_right_wheel"/>
-        <origin xyz="-0.15 -0.15 0" rpy="1.57079632679 0 0"/>
+        <origin xyz="-0.15 -0.15 0.05" rpy="0 0 0"/>
         <axis xyz="0 0 -1"/>
     </joint>
@@ -135,29 +124,5 @@
             </geometry>
         </collision>
-        <xacro:inertial_cylinder mass="0.1" length="0.04" radius="0.05">
-            <origin xyz="0 0 0" rpy="0 0 0"/>
-        </xacro:inertial_cylinder>
-    </link>
-    <!-- CASTER WHEEL (Optional) -->
-    <joint name="caster_wheel_joint" type="fixed">
-        <parent link="chassis"/>
-        <child link="caster_wheel"/>
-        <origin xyz="0.24 0 0"/>
-    </joint>
-    <link name="caster_wheel">
-        <visual>
-            <geometry>
-                <sphere radius="0.05"/>
-            </geometry>
-            <material name="black"/>
-        </visual>
-        <collision>
-            <geometry>
-                <sphere radius="0.05"/>
-            </geometry>
-        </collision>
-        <xacro:inertial_sphere mass="0.1" radius="0.05">
-            <origin xyz="0 0 0" rpy="0 0 0"></origin>
-        </xacro:inertial_sphere>
+        <xacro:inertial_cylinder mass="0.1" length="0.04" radius="0.05"/>
     </link>
 </robot>

Commit message: mecanum urdf fixes

File: src/main_sim/urdf/mecanum_core.xacro (robot description, xacro)
@@ -61,5 +61,7 @@
             </geometry>
         </collision>
-        <xacro:inertial_cylinder mass="0.1" length="0.04" radius="0.05"/>
+        <xacro:inertial_cylinder mass="0.1" length="0.04" radius="0.05">
+            <origin xyz="0 0 0" rpy="0 0 0"/>
+        </xacro:inertial_cylinder>
     </link>
     <!-- FRONT RIGHT WHEEL -->
@@ -82,5 +84,7 @@
             </geometry>
         </collision>
-        <xacro:inertial_cylinder mass="0.1" length="0.04" radius="0.05"/>
+        <xacro:inertial_cylinder mass="0.1" length="0.04" radius="0.05">
+            <origin xyz="0 0 0" rpy="0 0 0"/>
+        </xacro:inertial_cylinder>
     </link>
     <!-- REAR LEFT WHEEL -->
@@ -103,5 +107,7 @@
             </geometry>
         </collision>
-        <xacro:inertial_cylinder mass="0.1" length="0.04" radius="0.05"/>
+        <xacro:inertial_cylinder mass="0.1" length="0.04" radius="0.05">
+            <origin xyz="0 0 0" rpy="0 0 0"/>
+        </xacro:inertial_cylinder>
     </link>
     <!-- REAR RIGHT WHEEL -->
@@ -124,5 +130,7 @@
             </geometry>
         </collision>
-        <xacro:inertial_cylinder mass="0.1" length="0.04" radius="0.05"/>
+        <xacro:inertial_cylinder mass="0.1" length="0.04" radius="0.05">
+            <origin xyz="0 0 0" rpy="0 0 0"/>
+        </xacro:inertial_cylinder>
     </link>
 </robot>

File: src/main_sim/urdf/mecanum_inertial_macros.xacro (robot description, xacro)
@@ -1,5 +1,5 @@
 <?xml version="1.0"?>
 <robot xmlns:xacro="http://www.ros.org/xacro" >
-    <!-- Macro to define inertial properties for a box -->
+    <!-- Specify standard inertial calculations -->
     <xacro:macro name="inertial_box" params="mass x y z *origin">
         <inertial>
@@ -11,14 +11,7 @@
         </inertial>
     </xacro:macro>
-    <!-- Macro to define inertial properties for a cylinder -->
     <xacro:macro name="inertial_cylinder" params="mass length radius *origin">
         <inertial>
-            <!-- Ensure an origin is always included -->
-            <xacro:if value="${origin}">
-                <xacro:insert_block name="origin"/>
-            </xacro:if>
-            <xacro:unless value="${origin}">
-                <origin xyz="0 0 0" rpy="0 0 0"/>
-            </xacro:unless>
+            <xacro:insert_block name="origin"/>
             <mass value="${mass}" />
             <inertia ixx="${(1/12) * mass * (3*radius*radius + length*length)}" ixy="0.0" ixz="0.0"

Commit message: urdf updates

File: src/main_sim/urdf/mecanum_core.xacro (robot description, xacro)
@@ -46,5 +46,5 @@
         <parent link="base_link"/>
         <child link="front_left_wheel"/>
-        <origin xyz="0.15 0.15 0.05" rpy="0 0 0"/>
+        <origin xyz="0.15 0.175 0" rpy="1.5708 0 0"/>
         <axis xyz="0 0 1"/>
     </joint>
@@ -69,5 +69,5 @@
         <parent link="base_link"/>
         <child link="front_right_wheel"/>
-        <origin xyz="0.15 -0.15 0.05" rpy="0 0 0"/>
+        <origin xyz="0.15 -0.175 0" rpy="-1.5708 0 0"/>
         <axis xyz="0 0 -1"/>
     </joint>
@@ -92,5 +92,5 @@
         <parent link="base_link"/>
         <child link="rear_left_wheel"/>
-        <origin xyz="-0.15 0.15 0.05" rpy="0 0 0"/>
+        <origin xyz="-0.15 0.175 0" rpy="1.5708 0 0"/>
         <axis xyz="0 0 1"/>
     </joint>
@@ -115,5 +115,5 @@
         <parent link="base_link"/>
         <child link="rear_right_wheel"/>
-        <origin xyz="-0.15 -0.15 0.05" rpy="0 0 0"/>
+        <origin xyz="-0.15 -0.175 0" rpy="-1.5708 0 0"/>
         <axis xyz="0 0 -1"/>
     </joint>

File: src/main_sim/urdf/mecanum_robot.urdf.xacro (robot description, xacro)
@@ -1,4 +1,4 @@
 <?xml version="1.0"?>
-<robot xmlns:xacro="http://www.ros.org/wiki/xacro" name="robot">
+<robot xmlns:xacro="http://www.ros.org/xacro" name="robot">
     <xacro:include filename="mecanum_core.xacro" />
     <!-- <xacro:include filename="gazebo_control.xacro"/> -->

Commit message: urdf fixed

File: src/main_sim/urdf/mecanum_core.xacro (robot description, xacro)
@@ -46,5 +46,5 @@
         <parent link="base_link"/>
         <child link="front_left_wheel"/>
-        <origin xyz="0.15 0.175 0" rpy="1.5708 0 0"/>
+        <origin xyz="0.15 0.17 0" rpy="1.5708 0 0"/>
         <axis xyz="0 0 1"/>
     </joint>
@@ -69,5 +69,5 @@
         <parent link="base_link"/>
         <child link="front_right_wheel"/>
-        <origin xyz="0.15 -0.175 0" rpy="-1.5708 0 0"/>
+        <origin xyz="0.15 -0.17 0" rpy="-1.5708 0 0"/>
         <axis xyz="0 0 -1"/>
     </joint>
@@ -92,5 +92,5 @@
         <parent link="base_link"/>
         <child link="rear_left_wheel"/>
-        <origin xyz="-0.15 0.175 0" rpy="1.5708 0 0"/>
+        <origin xyz="-0.15 0.17 0" rpy="1.5708 0 0"/>
         <axis xyz="0 0 1"/>
     </joint>
@@ -115,5 +115,5 @@
         <parent link="base_link"/>
         <child link="rear_right_wheel"/>
-        <origin xyz="-0.15 -0.175 0" rpy="-1.5708 0 0"/>
+        <origin xyz="-0.15 -0.17 0" rpy="-1.5708 0 0"/>
         <axis xyz="0 0 -1"/>
     </joint>

Commit message: urdf changes

File: src/main_sim/urdf/mecanum_core.xacro (robot description, xacro)
@@ -46,5 +46,5 @@
         <parent link="base_link"/>
         <child link="front_left_wheel"/>
-        <origin xyz="0.15 0.17 0" rpy="1.5708 0 0"/>
+        <origin xyz="0.15 0.17 0" rpy="-1.5708 0 0"/>
         <axis xyz="0 0 1"/>
     </joint>
@@ -92,5 +92,5 @@
         <parent link="base_link"/>
         <child link="rear_left_wheel"/>
-        <origin xyz="-0.15 0.17 0" rpy="1.5708 0 0"/>
+        <origin xyz="-0.15 0.17 0" rpy="-1.5708 0 0"/>
         <axis xyz="0 0 1"/>
     </joint>

File: src/main_sim/urdf/mecanum_ros2_control.xacro (robot description, xacro)
@@ -44,5 +44,5 @@
     <gazebo>
         <plugin name="gz_ros2_control::GazeboSimROS2ControlPlugin" filename="libgz_ros2_control-system.so">
-            <parameters>src/main_sim/config/mecanum_control.yaml</parameters>
+            <parameters>/home/jason/ros2_ws/src/main_sim/config/mecanum_control.yaml</parameters>
             <parameters>/home/jason/ros2_ws/src/main_sim/config/ros_gz_ctrl_use_sim.yaml</parameters>
         </plugin>

Commit message: small tuning

File: src/main_sim/urdf/mecanum_core.xacro (robot description, xacro)
@@ -70,5 +70,5 @@
         <child link="front_right_wheel"/>
         <origin xyz="0.15 -0.17 0" rpy="-1.5708 0 0"/>
-        <axis xyz="0 0 -1"/>
+        <axis xyz="0 0 1"/>
     </joint>
     <link name="front_right_wheel">
@@ -116,5 +116,5 @@
         <child link="rear_right_wheel"/>
         <origin xyz="-0.15 -0.17 0" rpy="-1.5708 0 0"/>
-        <axis xyz="0 0 -1"/>
+        <axis xyz="0 0 1"/>
     </joint>
     <link name="rear_right_wheel">

Commit message: Update mecanum_core.xacro

File: src/main_sim/urdf/mecanum_core.xacro (robot description, xacro)
@@ -1,136 +1,192 @@
 <?xml version="1.0"?>
 <robot xmlns:xacro="http://www.ros.org/xacro">
-    <xacro:include filename="mecanum_inertial_macros.xacro"/>
-    <!-- Define Materials -->
-    <material name="white">
-        <color rgba="1 1 1 1"/>
-    </material>
-    <material name="blue">
-        <color rgba="0.2 0.2 1 1"/>
-    </material>
-    <!-- BASE LINK -->
-    <link name="base_link"/>
-    <!-- BASE_FOOTPRINT LINK -->
-    <joint name="base_footprint_joint" type="fixed">
-        <parent link="base_link"/>
-        <child link="base_footprint"/>
-        <origin xyz="0 0 0" rpy="0 0 0"/>
-    </joint>
-    <link name="base_footprint"/>
-    <!-- CHASSIS -->
-    <joint name="chassis_joint" type="fixed">
-        <parent link="base_link"/>
-        <child link="chassis"/>
-        <origin xyz="0 0 0"/>
-    </joint>
-    <link name="chassis">
-        <visual>
-            <origin xyz="0 0 0.075"/>
-            <geometry>
-                <box size="0.3 0.3 0.15"/>
-            </geometry>
-            <material name="white"/>
-        </visual>
-        <collision>
-            <origin xyz="0 0 0.075"/>
-            <geometry>
-                <box size="0.3 0.3 0.15"/>
-            </geometry>
-        </collision>
-        <xacro:inertial_box mass="0.5" x="0.3" y="0.3" z="0.15">
-            <origin xyz="0 0 0.075" rpy="0 0 0"/>
-        </xacro:inertial_box>
-    </link>
-    <!-- FRONT LEFT WHEEL -->
-    <joint name="front_left_wheel_joint" type="continuous">
-        <parent link="base_link"/>
-        <child link="front_left_wheel"/>
-        <origin xyz="0.15 0.17 0" rpy="-1.5708 0 0"/>
-        <axis xyz="0 0 1"/>
-    </joint>
-    <link name="front_left_wheel">
-        <visual>
-            <geometry>
-                <cylinder radius="0.05" length="0.04"/>
-            </geometry>
-            <material name="blue"/>
-        </visual>
-        <collision>
-            <geometry>
-                <cylinder radius="0.05" length="0.04"/>
-            </geometry>
-        </collision>
-        <xacro:inertial_cylinder mass="0.1" length="0.04" radius="0.05">
-            <origin xyz="0 0 0" rpy="0 0 0"/>
-        </xacro:inertial_cylinder>
-    </link>
-    <!-- FRONT RIGHT WHEEL -->
-    <joint name="front_right_wheel_joint" type="continuous">
-        <parent link="base_link"/>
-        <child link="front_right_wheel"/>
-        <origin xyz="0.15 -0.17 0" rpy="-1.5708 0 0"/>
-        <axis xyz="0 0 1"/>
-    </joint>
-    <link name="front_right_wheel">
-        <visual>
-            <geometry>
-                <cylinder radius="0.05" length="0.04"/>
-            </geometry>
-            <material name="blue"/>
-        </visual>
-        <collision>
-            <geometry>
-                <cylinder radius="0.05" length="0.04"/>
-            </geometry>
-        </collision>
-        <xacro:inertial_cylinder mass="0.1" length="0.04" radius="0.05">
-            <origin xyz="0 0 0" rpy="0 0 0"/>
-        </xacro:inertial_cylinder>
-    </link>
-    <!-- REAR LEFT WHEEL -->
-    <joint name="rear_left_wheel_joint" type="continuous">
-        <parent link="base_link"/>
-        <child link="rear_left_wheel"/>
-        <origin xyz="-0.15 0.17 0" rpy="-1.5708 0 0"/>
-        <axis xyz="0 0 1"/>
-    </joint>
-    <link name="rear_left_wheel">
-        <visual>
-            <geometry>
-                <cylinder radius="0.05" length="0.04"/>
-            </geometry>
-            <material name="blue"/>
-        </visual>
-        <collision>
-            <geometry>
-                <cylinder radius="0.05" length="0.04"/>
-            </geometry>
-        </collision>
-        <xacro:inertial_cylinder mass="0.1" length="0.04" radius="0.05">
-            <origin xyz="0 0 0" rpy="0 0 0"/>
-        </xacro:inertial_cylinder>
-    </link>
-    <!-- REAR RIGHT WHEEL -->
-    <joint name="rear_right_wheel_joint" type="continuous">
-        <parent link="base_link"/>
-        <child link="rear_right_wheel"/>
-        <origin xyz="-0.15 -0.17 0" rpy="-1.5708 0 0"/>
-        <axis xyz="0 0 1"/>
-    </joint>
-    <link name="rear_right_wheel">
-        <visual>
-            <geometry>
-                <cylinder radius="0.05" length="0.04"/>
-            </geometry>
-            <material name="blue"/>
-        </visual>
-        <collision>
-            <geometry>
-                <cylinder radius="0.05" length="0.04"/>
-            </geometry>
-        </collision>
-        <xacro:inertial_cylinder mass="0.1" length="0.04" radius="0.05">
-            <origin xyz="0 0 0" rpy="0 0 0"/>
-        </xacro:inertial_cylinder>
-    </link>
+  <xacro:include filename="mecanum_inertial_macros.xacro"/>
+  <!-- Define Materials -->
+  <material name="white">
+    <color rgba="1 1 1 1"/>
+  </material>
+  <material name="blue">
+    <color rgba="0.2 0.2 1 1"/>
+  </material>
+  <!-- BASE LINK -->
+  <link name="base_link"/>
+  <!-- BASE_FOOTPRINT LINK -->
+  <joint name="base_footprint_joint" type="fixed">
+    <parent link="base_link"/>
+    <child link="base_footprint"/>
+    <origin xyz="0 0 0" rpy="0 0 0"/>
+  </joint>
+  <link name="base_footprint"/>
+  <!-- CHASSIS -->
+  <joint name="chassis_joint" type="fixed">
+    <parent link="base_link"/>
+    <child link="chassis"/>
+    <origin xyz="0 0 0"/>
+  </joint>
+  <link name="chassis">
+    <visual>
+      <origin xyz="0 0 0.075"/>
+      <geometry>
+        <box size="0.3 0.3 0.15"/>
+      </geometry>
+      <material name="white"/>
+    </visual>
+    <collision>
+      <origin xyz="0 0 0.075"/>
+      <geometry>
+        <box size="0.3 0.3 0.15"/>
+      </geometry>
+    </collision>
+    <xacro:inertial_box mass="0.5" x="0.3" y="0.3" z="0.15">
+      <origin xyz="0 0 0.075" rpy="0 0 0"/>
+    </xacro:inertial_box>
+  </link>
+  <!-- FRONT LEFT WHEEL -->
+  <joint name="front_left_wheel_joint" type="continuous">
+    <parent link="base_link"/>
+    <child link="front_left_wheel"/>
+    <!--
+      rpy ~ -1.5708 means rotating the cylinder by -90 deg around X,
+      so the cylinder's axis is along Y.
+      Then the joint axis is <axis xyz="0 0 1"/>.
+    -->
+    <origin xyz="0.15 0.17 0" rpy="-1.5708 0 0"/>
+    <axis xyz="0 0 1"/>
+  </joint>
+  <link name="front_left_wheel">
+    <visual>
+      <geometry>
+        <cylinder radius="0.05" length="0.04"/>
+      </geometry>
+      <material name="blue"/>
+    </visual>
+    <collision>
+      <geometry>
+        <cylinder radius="0.05" length="0.04"/>
+      </geometry>
+      <!-- ADD FRICTION BLOCK -->
+      <surface>
+        <friction>
+          <ode>
+            <!--
+              mu = friction in fdir1, mu2 = friction perpendicular to fdir1.
+              For a typical front-left Mecanum wheel, let's guess fdir1>1 -1 0.
+              That means: high friction along the (1, -1, 0) diagonal, low friction sideways.
+            -->
+            <mu>1.0</mu>
+            <mu2>0.0</mu2>
+            <fdir1>1 -1 0</fdir1>
+          </ode>
+        </friction>
+      </surface>
+    </collision>
+    <xacro:inertial_cylinder mass="0.1" length="0.04" radius="0.05">
+      <origin xyz="0 0 0" rpy="0 0 0"/>
+    </xacro:inertial_cylinder>
+  </link>
+  <!-- FRONT RIGHT WHEEL -->
+  <joint name="front_right_wheel_joint" type="continuous">
+    <parent link="base_link"/>
+    <child link="front_right_wheel"/>
+    <origin xyz="0.15 -0.17 0" rpy="-1.5708 0 0"/>
+    <axis xyz="0 0 1"/>
+  </joint>
+  <link name="front_right_wheel">
+    <visual>
+      <geometry>
+        <cylinder radius="0.05" length="0.04"/>
+      </geometry>
+      <material name="blue"/>
+    </visual>
+    <collision>
+      <geometry>
+        <cylinder radius="0.05" length="0.04"/>
+      </geometry>
+      <!-- ADD FRICTION BLOCK -->
+      <surface>
+        <friction>
+          <ode>
+            <!-- For front-right, we might do fdir1>1 1 0 -->
+            <mu>1.0</mu>
+            <mu2>0.0</mu2>
+            <fdir1>1 1 0</fdir1>
+          </ode>
+        </friction>
+      </surface>
+    </collision>
+    <xacro:inertial_cylinder mass="0.1" length="0.04" radius="0.05">
+      <origin xyz="0 0 0" rpy="0 0 0"/>
+    </xacro:inertial_cylinder>
+  </link>
+  <!-- REAR LEFT WHEEL -->
+  <joint name="rear_left_wheel_joint" type="continuous">
+    <parent link="base_link"/>
+    <child link="rear_left_wheel"/>
+    <origin xyz="-0.15 0.17 0" rpy="-1.5708 0 0"/>
+    <axis xyz="0 0 1"/>
+  </joint>
+  <link name="rear_left_wheel">
+    <visual>
+      <geometry>
+        <cylinder radius="0.05" length="0.04"/>
+      </geometry>
+      <material name="blue"/>
+    </visual>
+    <collision>
+      <geometry>
+        <cylinder radius="0.05" length="0.04"/>
+      </geometry>
+      <!-- ADD FRICTION BLOCK -->
+      <surface>
+        <friction>
+          <ode>
+            <!--
+              For rear_left, might also be '1 1 0' or '1 -1 0'.
+              This depends on your roller orientation. Let's try 1 1 0 here.
+            -->
+            <mu>1.0</mu>
+            <mu2>0.0</mu2>
+            <fdir1>1 1 0</fdir1>
+          </ode>
+        </friction>
+      </surface>
+    </collision>
+    <xacro:inertial_cylinder mass="0.1" length="0.04" radius="0.05">
+      <origin xyz="0 0 0" rpy="0 0 0"/>
+    </xacro:inertial_cylinder>
+  </link>
+  <!-- REAR RIGHT WHEEL -->
+  <joint name="rear_right_wheel_joint" type="continuous">
+    <parent link="base_link"/>
+    <child link="rear_right_wheel"/>
+    <origin xyz="-0.15 -0.17 0" rpy="-1.5708 0 0"/>
+    <axis xyz="0 0 1"/>
+  </joint>
+  <link name="rear_right_wheel">
+    <visual>
+      <geometry>
+        <cylinder radius="0.05" length="0.04"/>
+      </geometry>
+      <material name="blue"/>
+    </visual>
+    <collision>
+      <geometry>
+        <cylinder radius="0.05" length="0.04"/>
+      </geometry>
+      <!-- ADD FRICTION BLOCK -->
+      <surface>
+        <friction>
+          <ode>
+            <!-- For rear-right, we might revert to '1 -1 0' again -->
+            <mu>1.0</mu>
+            <mu2>0.0</mu2>
+            <fdir1>1 -1 0</fdir1>
+          </ode>
+        </friction>
+      </surface>
+    </collision>
+    <xacro:inertial_cylinder mass="0.1" length="0.04" radius="0.05">
+      <origin xyz="0 0 0" rpy="0 0 0"/>
+    </xacro:inertial_cylinder>
+  </link>
 </robot>
