Commit message: temp testing

File: src/main_sim/urdf/mecanum_core.xacro (robot description, xacro)
@@ -38,5 +38,5 @@
       </geometry>
     </collision>
-    <xacro:inertial_box mass="0.5" x="0.3" y="0.3" z="0.15">
+    <xacro:inertial_box mass="4.0" x="0.3" y="0.3" z="0.15">
       <origin xyz="0 0 0.075" rpy="0 0 0"/>
     </xacro:inertial_box>
@@ -51,5 +51,5 @@
       Then the joint axis is <axis xyz="0 0 1"/>.
     -->
-    <origin xyz="0.15 0.17 0" rpy="-1.5708 0 0"/>
+    <origin xyz="0.15 0.17 0.025" rpy="-1.5708 0 0"/>
     <axis xyz="0 0 1"/>
   </joint>
@@ -81,5 +81,5 @@
       </surface>
     </collision>
-    <xacro:inertial_cylinder mass="0.1" length="0.04" radius="0.05">
+    <xacro:inertial_cylinder mass="1" length="0.04" radius="0.05">
       <origin xyz="0 0 0" rpy="0 0 0"/>
     </xacro:inertial_cylinder>
@@ -89,5 +89,5 @@
     <parent link="base_link"/>
     <child link="front_right_wheel"/>
-    <origin xyz="0.15 -0.17 0" rpy="-1.5708 0 0"/>
+    <origin xyz="0.15 -0.17 0.025" rpy="-1.5708 0 0"/>
     <axis xyz="0 0 1"/>
   </joint>
@@ -115,5 +115,5 @@
       </surface>
     </collision>
-    <xacro:inertial_cylinder mass="0.1" length="0.04" radius="0.05">
+    <xacro:inertial_cylinder mass="1" length="0.04" radius="0.05">
       <origin xyz="0 0 0" rpy="0 0 0"/>
     </xacro:inertial_cylinder>
@@ -123,5 +123,5 @@
     <parent link="base_link"/>
     <child link="rear_left_wheel"/>
-    <origin xyz="-0.15 0.17 0" rpy="-1.5708 0 0"/>
+    <origin xyz="-0.15 0.17 0.025" rpy="-1.5708 0 0"/>
     <axis xyz="0 0 1"/>
   </joint>
@@ -152,5 +152,5 @@
       </surface>
     </collision>
-    <xacro:inertial_cylinder mass="0.1" length="0.04" radius="0.05">
+    <xacro:inertial_cylinder mass="1" length="0.04" radius="0.05">
       <origin xyz="0 0 0" rpy="0 0 0"/>
     </xacro:inertial_cylinder>
@@ -160,5 +160,5 @@
     <parent link="base_link"/>
     <child link="rear_right_wheel"/>
-    <origin xyz="-0.15 -0.17 0" rpy="-1.5708 0 0"/>
+    <origin xyz="-0.15 -0.17 0.025" rpy="-1.5708 0 0"/>
     <axis xyz="0 0 1"/>
   </joint>
@@ -186,5 +186,5 @@
       </surface>
     </collision>
-    <xacro:inertial_cylinder mass="0.1" length="0.04" radius="0.05">
+    <xacro:inertial_cylinder mass="1" length="0.04" radius="0.05">
       <origin xyz="0 0 0" rpy="0 0 0"/>
     </xacro:inertial_cylinder>
