Commit message: new mecanum sphere urdf

File: src/main_sim/urdf/mecanum_sphere/mecanum_sphere_core.xacro (robot description, xacro)
@@ -1,5 +1,5 @@
 <?xml version="1.0"?>
 <robot xmlns:xacro="http://www.ros.org/xacro">
-  <xacro:include filename="mecanum_inertial_macros.xacro"/>
+  <xacro:include filename="inertial_macros_mecanum_sphere.xacro"/>
   <!-- Define Materials -->
   <material name="white">
@@ -46,9 +46,4 @@
     <parent link="base_link"/>
     <child link="front_left_wheel"/>
-    <!--
-      rpy ~ -1.5708 means rotating the cylinder by -90 deg around X,
-      so the cylinder's axis is along Y.
-      Then the joint axis is <axis xyz="0 0 1"/>.
-    -->
     <origin xyz="0.15 0.17 0.025" rpy="-1.5708 0 0"/>
     <axis xyz="0 0 1"/>

Commit message: Update mecanum_sphere_core.xacro

File: src/main_sim/urdf/mecanum_sphere/mecanum_sphere_core.xacro (robot description, xacro)
@@ -145,32 +145,31 @@
     <parent link="base_link"/>
     <child link="rear_right_wheel"/>
-    <origin xyz="-0.15 -0.17 0.025" rpy="-1.5708 0 0"/>
+    <origin xyz="-0.15 -0.17 0.025" rpy="0 0 0"/> <!-- No rotation needed for spheres -->
     <axis xyz="0 0 1"/>
   </joint>
-  <link name="rear_right_wheel">
-    <visual>
-      <geometry>
-        <cylinder radius="0.05" length="0.04"/>
-      </geometry>
-      <material name="blue"/>
-    </visual>
-    <collision>
-      <geometry>
-        <cylinder radius="0.05" length="0.04"/>
-      </geometry>
-      <!-- ADD FRICTION BLOCK -->
-      <!-- <surface>
-        <friction>
-          <ode>
-            <mu>1.0</mu>
-            <mu2>0.0</mu2>
-            <fdir1>1 -1 0</fdir1>
-          </ode>
-        </friction>
-      </surface> -->
-    </collision>
-    <xacro:inertial_cylinder mass="1" length="0.04" radius="0.05">
-      <origin xyz="0 0 0" rpy="0 0 0"/>
-    </xacro:inertial_cylinder>
-  </link>
+<link name="rear_right_wheel">
+  <visual>
+    <geometry>
+      <sphere radius="0.05"/>
+    </geometry>
+    <material name="blue"/>
+  </visual>
+  <collision>
+    <geometry>
+      <sphere radius="0.05"/>
+    </geometry>
+    <surface>
+      <friction>
+        <ode>
+          <mu>1.0</mu>
+          <mu2>0.0</mu2>
+          <fdir1>1 -1 0</fdir1>
+        </ode>
+      </friction>
+    </surface>
+  </collision>
+  <xacro:inertial_sphere mass="1" radius="0.05">
+    <origin xyz="0 0 0" rpy="0 0 0"/>
+  </xacro:inertial_sphere>
+</link>
 </robot>

Commit message: mecanum sphere

File: src/main_sim/urdf/mecanum_sphere/mecanum_sphere_core.xacro (robot description, xacro)
@@ -38,5 +38,5 @@
       </geometry>
     </collision>
-    <xacro:inertial_box mass="4.0" x="0.3" y="0.3" z="0.15">
+    <xacro:inertial_box mass="6.0" x="0.3" y="0.3" z="0.15">
       <origin xyz="0 0 0.075" rpy="0 0 0"/>
     </xacro:inertial_box>
@@ -52,5 +52,5 @@
     <visual>
       <geometry>
-        <cylinder radius="0.05" length="0.04"/>
+        <sphere radius="0.05"/>
       </geometry>
       <material name="blue"/>
@@ -58,8 +58,7 @@
     <collision>
       <geometry>
-        <cylinder radius="0.05" length="0.04"/>
+        <sphere radius="0.05"/>
       </geometry>
-      <!-- ADD FRICTION BLOCK -->
-      <!-- <surface>
+      <surface>
         <friction>
           <ode>
@@ -69,9 +68,9 @@
           </ode>
         </friction>
-      </surface> -->
+      </surface>
     </collision>
-    <xacro:inertial_cylinder mass="1" length="0.04" radius="0.05">
+    <xacro:inertial_sphere mass="1" radius="0.05">
       <origin xyz="0 0 0" rpy="0 0 0"/>
-    </xacro:inertial_cylinder>
+    </xacro:inertial_sphere>
   </link>
   <!-- FRONT RIGHT WHEEL -->
@@ -85,5 +84,5 @@
     <visual>
       <geometry>
-        <cylinder radius="0.05" length="0.04"/>
+        <sphere radius="0.05"/>
       </geometry>
       <material name="blue"/>
@@ -91,8 +90,7 @@
     <collision>
       <geometry>
-        <cylinder radius="0.05" length="0.04"/>
+        <sphere radius="0.05"/>
       </geometry>
-      <!-- ADD FRICTION BLOCK -->
-      <!-- <surface>
+      <surface>
         <friction>
           <ode>
@@ -102,9 +100,9 @@
           </ode>
         </friction>
-      </surface> -->
+      </surface>
     </collision>
-    <xacro:inertial_cylinder mass="1" length="0.04" radius="0.05">
+    <xacro:inertial_sphere mass="1" radius="0.05">
       <origin xyz="0 0 0" rpy="0 0 0"/>
-    </xacro:inertial_cylinder>
+    </xacro:inertial_sphere>
   </link>
   <!-- REAR LEFT WHEEL -->
@@ -118,5 +116,5 @@
     <visual>
       <geometry>
-        <cylinder radius="0.05" length="0.04"/>
+        <sphere radius="0.05"/>
       </geometry>
       <material name="blue"/>
@@ -124,8 +122,7 @@
     <collision>
       <geometry>
-        <cylinder radius="0.05" length="0.04"/>
+        <sphere radius="0.05"/>
       </geometry>
-      <!-- ADD FRICTION BLOCK -->
-      <!-- <surface>
+      <surface>
         <friction>
           <ode>
@@ -135,9 +132,9 @@
           </ode>
         </friction>
-      </surface> -->
+      </surface>
     </collision>
-    <xacro:inertial_cylinder mass="1" length="0.04" radius="0.05">
+    <xacro:inertial_sphere mass="1" radius="0.05">
       <origin xyz="0 0 0" rpy="0 0 0"/>
-    </xacro:inertial_cylinder>
+    </xacro:inertial_sphere>
   </link>
   <!-- REAR RIGHT WHEEL -->
@@ -145,5 +142,5 @@
     <parent link="base_link"/>
     <child link="rear_right_wheel"/>
-    <origin xyz="-0.15 -0.17 0.025" rpy="0 0 0"/> <!-- No rotation needed for spheres -->
+    <origin xyz="-0.15 -0.17 0.025" rpy="-1.5708 0 0"/> <!-- No rotation needed for spheres -->
     <axis xyz="0 0 1"/>
   </joint>

Commit message: added correct friction hopefully

File: src/main_sim/urdf/mecanum_sphere/mecanum_sphere_core.xacro (robot description, xacro)
@@ -156,13 +156,4 @@
       <sphere radius="0.05"/>
     </geometry>
-    <surface>
-      <friction>
-        <ode>
-          <mu>1.0</mu>
-          <mu2>0.01</mu2>
-          <fdir1>-1 -1 0</fdir1>
-        </ode>
-      </friction>
-    </surface>
   </collision>
   <xacro:inertial_sphere mass="1" radius="0.05">
@@ -170,3 +161,55 @@
   </xacro:inertial_sphere>
 </link>
+<gazebo reference='front_left_wheel'>
+    <collision>
+      <surface>
+        <friction>
+          <ode>
+            <mu>1.0</mu>
+            <mu2>0.0</mu2>
+            <fdir1 gz:expressed_in="base_link">1 -1 0</fdir1>
+          </ode>
+        </friction>
+      </surface>
+    </collision>
+  </gazebo>
+  <gazebo reference='front_right_wheel'>
+    <collision>
+      <surface>
+        <friction>
+          <ode>
+            <mu>1.0</mu>
+            <mu2>0.0</mu2>
+            <fdir1 gz:expressed_in="base_link">1 1 0</fdir1>
+          </ode>
+        </friction>
+      </surface>
+    </collision>
+  </gazebo>
+  <gazebo reference='rear_left_wheel'>
+    <collision>
+      <surface>
+        <friction>
+          <ode>
+            <mu>1.0</mu>
+            <mu2>0.0</mu2>
+            <fdir1 gz:expressed_in="base_link">1 1 0</fdir1>
+          </ode>
+        </friction>
+      </surface>
+    </collision>
+  </gazebo>
+  <gazebo reference='rear_right_wheel'>
+    <collision>
+      <surface>
+        <friction>
+          <ode>
+            <mu>1.0</mu>
+            <mu2>0.0</mu2>
+            <fdir1 gz:expressed_in="base_link">1 -1 0</fdir1>
+          </ode>
+        </friction>
+      </surface>
+    </collision>
+  </gazebo>
 </robot>

Commit message: STRAFING WORKS

File: src/main_sim/urdf/mecanum_sphere/mecanum_sphere_core.xacro (robot description, xacro)
@@ -1,4 +1,5 @@
 <?xml version="1.0"?>
-<robot xmlns:xacro="http://www.ros.org/xacro">
+<robot xmlns:xacro="http://www.ros.org/xacro"
+      xmlns:gz="http://gazebosim.org/schema">
   <xacro:include filename="inertial_macros_mecanum_sphere.xacro"/>
   <!-- Define Materials -->
@@ -60,13 +61,4 @@
         <sphere radius="0.05"/>
       </geometry>
-      <surface>
-        <friction>
-          <ode>
-            <mu>1.0</mu>
-            <mu2>0.01</mu2>
-            <fdir1>1 1 0</fdir1>
-          </ode>
-        </friction>
-      </surface>
     </collision>
     <xacro:inertial_sphere mass="1" radius="0.05">
@@ -92,13 +84,4 @@
         <sphere radius="0.05"/>
       </geometry>
-      <surface>
-        <friction>
-          <ode>
-            <mu>1.0</mu>
-            <mu2>0.01</mu2>
-            <fdir1>1 -1 0</fdir1>
-          </ode>
-        </friction>
-      </surface>
     </collision>
     <xacro:inertial_sphere mass="1" radius="0.05">
@@ -123,14 +106,5 @@
       <geometry>
         <sphere radius="0.05"/>
-      </geometry>
-      <surface>
-        <friction>
-          <ode>
-            <mu>1.0</mu>
-            <mu2>0.01</mu2>
-            <fdir1>-1 1 0</fdir1>
-          </ode>
-        </friction>
-      </surface>
+      </geometry>>
     </collision>
     <xacro:inertial_sphere mass="1" radius="0.05">
@@ -161,5 +135,5 @@
   </xacro:inertial_sphere>
 </link>
-<gazebo reference='front_left_wheel'>
+  <gazebo reference='front_left_wheel'>
     <collision>
       <surface>
