Commit message: working on lidar now

File: src/main_sim/urdf/mecanum_sphere/inertial_macros_mecanum_sphere.xacro (robot description, xacro)
@@ -21,3 +21,12 @@
         </inertial>
     </xacro:macro>
+    <xacro:macro name="inertial_cylinder" params="mass length radius *origin">
+        <inertial>
+            <xacro:insert_block name="origin"/>
+            <mass value="${mass}" />
+            <inertia ixx="${(1/12) * mass * (3*radius*radius + length*length)}" ixy="0.0" ixz="0.0"
+                    iyy="${(1/12) * mass * (3*radius*radius + length*length)}" iyz="0.0"
+                    izz="${(1/2) * mass * (radius*radius)}" />
+        </inertial>
+    </xacro:macro>
 </robot>

File: src/main_sim/urdf/mecanum_sphere/mecanum_sphere.urdf.xacro (robot description, xacro)
@@ -4,4 +4,4 @@
     <!-- <xacro:include filename="gazebo_control.xacro"/> -->
     <xacro:include filename="ros2_control_mecanum_sphere.xacro"/>
-    <!-- <xacro:include filename="lidar.xacro"/> -->
+    <xacro:include filename="mecanum_lidar.xacro"/>
 </robot>

File: src/main_sim/urdf/mecanum_sphere/ros2_control_mecanum_sphere.xacro (robot description, xacro)
@@ -48,5 +48,6 @@
             <ros>
                 <remapping>/mecanum_cont/reference:=/cmd_vel</remapping>
-                <remapping>/mecanum_cont/odom:=/odom</remapping>
+                <remapping>/mecanum_cont/odometry:=/odom</remapping>
+                <remapping>/mecanum_cont/tf_odometry:=/tf</remapping>
             </ros>
         </plugin>
