Commit message: lidar tuning

File: src/main_sim/urdf/mecanum_sphere/mecanum_lidar.xacro (robot description, xacro)
@@ -1,5 +1,4 @@
 <?xml version="1.0"?>
 <robot xmlns:xacro="http://www.ros.org/wiki/xacro">
-    <xacro:include filename="inertial_macros_mecanum_sphere.xacro"/>
     <joint name="laser_joint" type="fixed">
         <parent link="chassis"/>

File: src/main_sim/urdf/mecanum_sphere/mecanum_sphere_core.xacro (robot description, xacro)
@@ -5,9 +5,18 @@
   <!-- Define Materials -->
   <material name="white">
-    <color rgba="1 1 1 1"/>
-  </material>
-  <material name="blue">
-    <color rgba="0.2 0.2 1 1"/>
-  </material>
+        <color rgba="1 1 1 1" />
+    </material>
+    <material name="orange">
+        <color rgba="1 0.3 0.1 1"/>
+    </material>
+    <material name="blue">
+        <color rgba="0.2 0.2 1 1"/>
+    </material>
+    <material name="black">
+        <color rgba="0 0 0 1"/>
+    </material>
+    <material name="red">
+        <color rgba="1 0 0 1"></color>
+    </material>
   <!-- BASE LINK -->
   <link name="base_link"/>
